File: PCB Files/TKL.sch (KiCad schematic (older format))
At the start: 227 parts, among them J1 USB_C, SW1 ESC, SW10 F9, SW100 RGUI_R2, SW101 RCTRL_R2, SW102 STEPPED_CAPS, SW103 RSHFT_175, SW104 Fn, SW105 BKSP_2U, SW11 F10, SW12 F11, SW13 F12, SW14 PRTSC, SW15 SCRLCK, SW16 PAUSE, SW17 GRV, SW18 1, SW19 2, SW2 F1, SW20 3, SW21 4, SW22 5, SW23 6, SW24 7, SW25 8, SW26 9, SW27 0, SW28 HIFEN, SW29 PLUS, SW3 F2, SW30 BCKSLSH, SW31 DEL, SW32 INS, SW33 HOME, SW34 PGUP, SW35 TAB, SW36 Q, SW37 W, SW38 E, SW39 R, SW4 F3, SW40 T, SW41 Y, SW42 U, SW43 I, SW44 O, SW45 P, SW46 LBRACES, SW47 RBRACES, SW48 BKSP_150, SW49 DEL, SW5 F4, SW50 END, SW51 PGDN, SW52 CAPS, SW53 A, SW54 S, SW55 D, SW56 F, SW57 G, SW58 H, SW59 J, SW6 F5, SW60 K, SW61 L, SW62 :, SW63 QUOTE, SW64 ENTER, SW65 LSHFT, SW66 Z, SW67 X, SW68 C, SW69 V, SW7 F6, SW70 B, SW71 N, SW72 M, SW73 <,, SW74 .>, SW75 /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

Commit message: Positioned switches
- The switches were positioned onto the PCB and the first WS2811 modules and RGB LEDs also were added. As of this commit, the edge layer drawings are a simple guideline and won't reflect the final dimensions or format.

- Added plated logo
Parts:
- added RGB2, RGB3, RGB4, RGB5, RGB6, RGB7: E6C1209RGB, acheron_Components:LED_RGB_SMD_6028_2.8x3.5mm_Round, symbol acheronSymbols:LED_GBRA
- added U2, U3, U4, U5, U6, U7: WS2811M, acheron_Components:MSOP-8-1EP_3x3mm_P0.65mm_EP1.68x1.88mm, symbol Driver_LED:WS2811
- RGB1: footprint acheron_Components:E6C1209RGB -> acheron_Components:LED_RGB_SMD_6028_2.8x3.5mm_Round
Connections:
- net 5V: now also RGB2.4 (A), RGB3.4 (A), RGB4.4 (A), RGB5.4 (A), RGB6.4 (A), RGB7.4 (A), U2.8 (VDD), U3.8 (VDD), U4.8 (VDD), U5.8 (VDD), U6.8 (VDD), U7.8 (VDD)
- net GND: now also U2.4 (GND), U3.4 (GND), U4.4 (GND), U5.4 (GND), U6.4 (GND), U7.4 (GND)
- new net: RGB2.1 (GK), U2.2 (OUTG)
- new net: RGB2.2 (BK), U2.3 (OUTB)
- new net: RGB2.3 (RK), U2.1 (OUTR)
- new net: RGB3.1 (GK), U3.2 (OUTG)
- new net: RGB3.2 (BK), U3.3 (OUTB)
- new net: RGB3.3 (RK), U3.1 (OUTR)
- new net: RGB4.1 (GK), U4.2 (OUTG)
- new net: RGB4.2 (BK), U4.3 (OUTB)
- new net: RGB4.3 (RK), U4.1 (OUTR)
- new net: RGB5.1 (GK), U5.2 (OUTG)
- new net: RGB5.2 (BK), U5.3 (OUTB)
- new net: RGB5.3 (RK), U5.1 (OUTR)
- new net: RGB6.1 (GK), U6.2 (OUTG)
- new net: RGB6.2 (BK), U6.3 (OUTB)
- new net: RGB6.3 (RK), U6.1 (OUTR)
- new net: RGB7.1 (GK), U7.2 (OUTG)
- new net: RGB7.2 (BK), U7.3 (OUTB)
- new net: RGB7.3 (RK), U7.1 (OUTR)
Other:
- moved on the sheet: RGB1, U1

Commit message: Routed RGB components and reorganized columns
- The WS2811M datasheet states that every unit must have two resistors and a capacitor around it; one resistor (33R) for the data lines and a resistor and capacitor (RC filter, 100R and 100nF) for bypass and spike prevention. These components were added.
- Laid the RGB components for some switches. Following the addition of the extra components for the RGB controllers, the RGB components (controller, resistors and capacitor and the LED) were added to a fourth of the total switches. The trace pattern was made to be repeatable through the whole PCB, in order to make a somewhat default trace pattern.
- The bigger 15x21mm short Acheron logo was added.
- Some switches had their columns reassigned for a better trace pattern. Some reorganizing should still be done in the future as the columns are traced.
Parts:
- removed RGB1, RGB2, RGB3, RGB4, RGB5, RGB6, RGB7: E6C1209RGB, acheron_Components:LED_RGB_SMD_6028_2.8x3.5mm_Round, symbol acheronSymbols:LED_GBRA
- added C1, C10, C11, C12, C13, C14, C15, C16, C2, C28, C29, C3, C30, C31, C32, C33, C34, C4, C5, C6, C7, C8, C9: 100nF, Capacitor_SMD:C_0805_2012Metric, symbol Device:C_Small
- added L1, L10, L11, L12, L13, L14, L15, L16, L2, L28, L29, L3, L30, L31, L32, L33, L34, L4, L5, L6, L7, L8, L9: LED_BGRA, acheron_Components:LED_RGB_SMD_6028_2.8x3.5mm_Round, symbol Device:LED_BGRA
- added R1, R10, R11, R12, R13, R14, R15, R16, R2, R28, R29, R3, R30, R31, R32, R33, R34, R4, R5, R6, R7, R8, R9: 100R, Resistor_SMD:R_0805_2012Metric, symbol Device:R_Small
- added RD1, RD10, RD11, RD12, RD13, RD14, RD15, RD16, RD2, RD28, RD29, RD3, RD30, RD31, RD33, RD34, RD4, RD5, RD6, RD7, RD8, RD9: 33R, Resistor_SMD:R_0805_2012Metric, symbol Device:R_Small
- added U10, U11, U12, U13, U14, U15, U16, U28, U29, U30, U31, U32, U33, U34, U8, U9: WS2811M, acheron_Components:MSOP-8-1EP_3x3mm_P0.65mm_EP1.68x1.88mm, symbol acheronSymbols:WS2811M
- U1, U2, U3, U4, U5, U6, U7: symbol Driver_LED:WS2811 -> acheronSymbols:WS2811M
- renumbered L1 to G1, L2 to G2, U29 to U200, U28 to U201
Connections:
- net 5V: now also L1.4 (A), L10.4 (A), L11.4 (A), L12.4 (A), L13.4 (A), L14.4 (A), L15.4 (A), L16.4 (A), L2.4 (A), L28.4 (A), L29.4 (A), L3.4 (A), L30.4 (A), L31.4 (A), L32.4 (A), L33.4 (A), L34.4 (A), L4.4 (A), L5.4 (A), L6.4 (A), L7.4 (A), L8.4 (A), L9.4 (A), R1.1, R10.1, R11.1, R12.1, R13.1, R14.1, R15.1, R16.1, R2.1, R28.1, R29.1, R3.1, R30.1, R31.1, R32.1, R33.1, R34.1, R4.1, R5.1, R6.1, R7.1, R8.1, R9.1; no longer U1.8 (VDD), U2.8 (VDD), U3.8 (VDD), U4.8 (VDD), U5.8 (VDD), U6.8 (VDD), U7.8 (VDD)
- net Col12: no longer SW103.1 (Col), SW63.1 (Col), SW76.1 (Col)
- net Col13: now also SW103.1 (Col), SW63.1 (Col), SW76.1 (Col); no longer SW101.1 (Col), SW104.1 (Col), SW64.1 (Col), SW85.1 (Col)
- net Col14: no longer SW48.1 (Col)
- net Col15: now also SW101.1 (Col), SW104.1 (Col), SW48.1 (Col), SW64.1 (Col), SW85.1 (Col)
- net GND: now also U1.9 (GND), U2.9 (GND), U3.9 (GND), U4.9 (GND), U5.9 (GND), U6.9 (GND), U7.9 (GND), C1.2, C10.2, C11.2, C12.2, C13.2, C14.2, C15.2, C16.2, C2.2, C28.2, C29.2, C3.2, C30.2, C31.2, C32.2, C33.2, C34.2, C4.2, C5.2, C6.2, C7.2, C8.2, C9.2, U10.4 (GND), U10.9 (GND), U11.4 (GND), U11.9 (GND), U12.4 (GND), U12.9 (GND), U13.4 (GND), U13.9 (GND), U14.4 (GND), U14.9 (GND), U15.4 (GND), U15.9 (GND), U16.4 (GND), U16.9 (GND), U28.4 (GND), U28.9 (GND), U29.4 (GND), U29.9 (GND), U30.4 (GND), U30.9 (GND), U31.4 (GND), U31.9 (GND), U32.4 (GND), U32.9 (GND), U33.4 (GND), U33.9 (GND), U34.4 (GND), U34.9 (GND), U8.4 (GND), U8.9 (GND), U9.4 (GND), U9.9 (GND)
- net at U1.1 (OUTR): now also L1.3 (RK)
- net at U1.2 (OUTG): now also L1.2 (GK)
- net at U1.3 (OUTB): now also L1.1 (BK)
- net at U1.5 (DO): now also RD1.2
- net at U2.2 (OUTG): now also L2.2 (GK)
- net at U2.3 (OUTB): now also L2.1 (BK)
- net at U2.1 (OUTR): now also L2.3 (RK)
- net at U2.5 (DO): now also RD2.2
- net at U2.6 (DIN): now also RD1.1
- net at U3.2 (OUTG): now also L3.2 (GK)
- net at U3.3 (OUTB): now also L3.1 (BK)
- net at U3.1 (OUTR): now also L3.3 (RK)
- net at U3.5 (DO): now also RD3.2
- net at U3.6 (DIN): now also RD2.1
- net at U4.2 (OUTG): now also L4.2 (GK)
- net at U4.3 (OUTB): now also L4.1 (BK)
- net at U4.1 (OUTR): now also L4.3 (RK)
- net at U4.5 (DO): now also RD4.2
- net at U4.6 (DIN): now also RD3.1
- net at U5.2 (OUTG): now also L5.2 (GK)
- net at U5.3 (OUTB): now also L5.1 (BK)
- net at U5.1 (OUTR): now also L5.3 (RK)
- net at U5.5 (DO): now also RD5.2
- net at U5.6 (DIN): now also RD4.1
- net at U6.2 (OUTG): now also L6.2 (GK)
- net at U6.3 (OUTB): now also L6.1 (BK)
- net at U6.1 (OUTR): now also L6.3 (RK)
- net at U6.5 (DO): now also RD6.2
- net at U6.6 (DIN): now also RD5.1
- net at U7.2 (OUTG): now also L7.2 (GK)
- net at U7.3 (OUTB): now also L7.1 (BK)
- net at U7.1 (OUTR): now also L7.3 (RK)
- net at U7.5 (DO): now also RD7.2
- net at U7.6 (DIN): now also RD6.1
- new net: C1.1, R1.2, U1.8 (VDD)
- new net: C2.1, R2.2, U2.8 (VDD)
- new net: C3.1, R3.2, U3.8 (VDD)
- new net: C4.1, R4.2, U4.8 (VDD)
- new net: C5.1, R5.2, U5.8 (VDD)
- new net: C6.1, R6.2, U6.8 (VDD)
- new net: C7.1, R7.2, U7.8 (VDD)
- new net: L8.3 (RK), U8.1 (OUTR)
- new net: L8.2 (GK), U8.2 (OUTG)
- new net: L8.1 (BK), U8.3 (OUTB)
- new net: RD8.2, U8.5 (DO)
- new net: RD7.1, U8.6 (DIN)
- new net: C8.1, R8.2, U8.8 (VDD)
- new net: L34.3 (RK), U34.1 (OUTR)
- new net: L34.2 (GK), U34.2 (OUTG)
- new net: L34.1 (BK), U34.3 (OUTB)
- new net: RD34.2, U34.5 (DO)
- new net: RD16.1, U34.6 (DIN)
- new net: C34.1, R34.2, U34.8 (VDD)
- new net: RD34.1, U33.6 (DIN)
- new net: L9.3 (RK), U9.1 (OUTR)
- new net: L9.2 (GK), U9.2 (OUTG)
- new net: L9.1 (BK), U9.3 (OUTB)
- new net: RD9.2, U9.5 (DO)
- new net: RD8.1, U9.6 (DIN)
- new net: C9.1, R9.2, U9.8 (VDD)
- new net: L10.3 (RK), U10.1 (OUTR)
- new net: L10.2 (GK), U10.2 (OUTG)
- new net: L10.1 (BK), U10.3 (OUTB)
- new net: RD10.2, U10.5 (DO)
- new net: RD9.1, U10.6 (DIN)
- new net: C10.1, R10.2, U10.8 (VDD)
- new net: L11.3 (RK), U11.1 (OUTR)
- new net: L11.2 (GK), U11.2 (OUTG)
- new net: L11.1 (BK), U11.3 (OUTB)
- new net: RD11.2, U11.5 (DO)
- new net: RD10.1, U11.6 (DIN)
- new net: C11.1, R11.2, U11.8 (VDD)
- new net: L12.3 (RK), U12.1 (OUTR)
- new net: L12.2 (GK), U12.2 (OUTG)
- new net: L12.1 (BK), U12.3 (OUTB)
- new net: RD12.2, U12.5 (DO)
- new net: RD11.1, U12.6 (DIN)
- new net: C12.1, R12.2, U12.8 (VDD)
- new net: L33.3 (RK), U33.1 (OUTR)
- new net: L33.2 (GK), U33.2 (OUTG)
- new net: L33.1 (BK), U33.3 (OUTB)
- new net: RD33.2, U33.5 (DO)
- new net: C33.1, R33.2, U33.8 (VDD)
- new net: RD33.1, U32.6 (DIN)
- new net: L32.3 (RK), U32.1 (OUTR)
- new net: L32.2 (GK), U32.2 (OUTG)
- new net: L32.1 (BK), U32.3 (OUTB)
- new net: RD31.2, U32.5 (DO)
- new net: C32.1, R32.2, U32.8 (VDD)
- new net: RD31.1, U31.6 (DIN)
- new net: L31.3 (RK), U31.1 (OUTR)
- new net: L31.2 (GK), U31.2 (OUTG)
- new net: L31.1 (BK), U31.3 (OUTB)
- new net: RD30.2, U31.5 (DO)
- new net: C31.1, R31.2, U31.8 (VDD)
- new net: RD30.1, U30.6 (DIN)
- new net: L30.3 (RK), U30.1 (OUTR)
- new net: L30.2 (GK), U30.2 (OUTG)
- new net: L30.1 (BK), U30.3 (OUTB)
- new net: RD29.2, U30.5 (DO)
- new net: C30.1, R30.2, U30.8 (VDD)
- new net: RD12.1, U13.6 (DIN)
- new net: L13.3 (RK), U13.1 (OUTR)
- new net: L13.2 (GK), U13.2 (OUTG)
- new net: L13.1 (BK), U13.3 (OUTB)
- new net: RD13.2, U13.5 (DO)
- new net: C13.1, R13.2, U13.8 (VDD)
- new net: RD13.1, U14.6 (DIN)
- new net: L14.3 (RK), U14.1 (OUTR)
- new net: L14.2 (GK), U14.2 (OUTG)
- new net: L14.1 (BK), U14.3 (OUTB)
- new net: RD14.2, U14.5 (DO)
- new net: C14.1, R14.2, U14.8 (VDD)
- new net: RD14.1, U15.6 (DIN)
- new net: L15.3 (RK), U15.1 (OUTR)
- new net: L15.2 (GK), U15.2 (OUTG)
- new net: L15.1 (BK), U15.3 (OUTB)
- new net: RD15.2, U15.5 (DO)
- new net: C15.1, R15.2, U15.8 (VDD)
- new net: RD15.1, U16.6 (DIN)
- new net: L16.3 (RK), U16.1 (OUTR)
- new net: L16.2 (GK), U16.2 (OUTG)
- new net: L16.1 (BK), U16.3 (OUTB)
- new net: RD16.2, U16.5 (DO)
- new net: C16.1, R16.2, U16.8 (VDD)
- new net: RD29.1, U29.6 (DIN)
- new net: L29.3 (RK), U29.1 (OUTR)
- new net: L29.2 (GK), U29.2 (OUTG)
- new net: L29.1 (BK), U29.3 (OUTB)
- new net: RD28.2, U29.5 (DO)
- new net: C29.1, R29.2, U29.8 (VDD)
- new net: RD28.1, U28.6 (DIN)
- new net: L28.3 (RK), U28.1 (OUTR)
- new net: L28.2 (GK), U28.2 (OUTG)
- new net: L28.1 (BK), U28.3 (OUTB)
- new net: C28.1, R28.2, U28.8 (VDD)
Other:
- moved on the sheet: D48, D63, D64, D76, D85, D90, SW101, SW103, SW104, SW48, SW63, SW64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

Commit message: Further routing and placement
Parts:
- removed RD16: 33R, Resistor_SMD:R_0805_2012Metric, symbol Device:R_Small
- added C17, C18, C19, C20, C21, C22, C23, C24, C25, C26, C27, C28: 100nF, Capacitor_SMD:C_0805_2012Metric, symbol Device:C_Small
- added L17, L18, L19, L20, L21, L22, L23, L24, L25, L26, L27, L28: LED_BGRA, acheron_Components:LED_RGB_SMD_6028_2.8x3.5mm_Round, symbol Device:LED_BGRA
- added R17, R18, R19, R20, R21, R22, R23, R24, R25, R26, R27, R28: 100R, Resistor_SMD:R_0805_2012Metric, symbol Device:R_Small
- added RD1, RD18, RD19, RD20, RD21, RD22, RD23, RD24, RD25, RD26, RD27, RD28, RD29: 33R, Resistor_SMD:R_0805_2012Metric, symbol Device:R_Small
- added U17, U18, U19, U20, U21, U22, U23, U24, U25, U26, U27, U28: WS2811M, acheron_Components:MSOP-8-1EP_3x3mm_P0.65mm_EP1.68x1.88mm, symbol acheronSymbols:WS2811M
- G2: footprint acheron_Logos:acheronShort_0.3x0.5in_Plated -> acheron_Logos:acheronShort_15.2x21mm_Plated
- renumbered C30 to C105, C28 to C29, C29 to C30, L30 to L105, L28 to L29, L29 to L30, R30 to R105, R28 to R29, R29 to R30, RD9 to RD10, RD29 to RD105, RD10 to RD11, RD11 to RD12, RD12 to RD13, RD13 to RD14, RD14 to RD15, RD15 to RD16, RD1 to RD2, RD2 to RD3, RD28 to RD30, RD30 to RD31, RD31 to RD32, RD3 to RD4, RD4 to RD5, RD5 to RD6, RD6 to RD7, RD7 to RD8, RD8 to RD9, U30 to U105, U28 to U29, U29 to U30
Connections:
- net 5V: now also L17.4 (A), L18.4 (A), L19.4 (A), L20.4 (A), L21.4 (A), L22.4 (A), L23.4 (A), L24.4 (A), L25.4 (A), L26.4 (A), L27.4 (A), L28.4 (A), R17.1, R18.1, R19.1, R20.1, R21.1, R22.1, R23.1, R24.1, R25.1, R26.1, R27.1, R28.1
- net GND: now also C17.2, C18.2, C19.2, C20.2, C21.2, C22.2, C23.2, C24.2, C25.2, C26.2, C27.2, C28.2, U17.4 (GND), U17.9 (GND), U18.4 (GND), U18.9 (GND), U19.4 (GND), U19.9 (GND), U20.4 (GND), U20.9 (GND), U21.4 (GND), U21.9 (GND), U22.4 (GND), U22.9 (GND), U23.4 (GND), U23.9 (GND), U24.4 (GND), U24.9 (GND), U25.4 (GND), U25.9 (GND), U26.4 (GND), U26.9 (GND), U27.4 (GND), U27.9 (GND), U28.4 (GND), U28.9 (GND)
- net RGB_DIN: now also RD1.2; no longer U1.6 (DIN)
- net at U29.5 (DO): now also RD29.2
- new net: RD1.1, U1.6 (DIN)
- new net: RD18.1, U17.6 (DIN)
- new net: RD18.2, U18.5 (DO)
- new net: L17.3 (RK), U17.1 (OUTR)
- new net: L17.2 (GK), U17.2 (OUTG)
- new net: L17.1 (BK), U17.3 (OUTB)
- new net: C17.1, R17.2, U17.8 (VDD)
- new net: RD19.1, U18.6 (DIN)
- new net: RD19.2, U19.5 (DO)
- new net: L18.3 (RK), U18.1 (OUTR)
- new net: L18.2 (GK), U18.2 (OUTG)
- new net: L18.1 (BK), U18.3 (OUTB)
- new net: C18.1, R18.2, U18.8 (VDD)
- new net: RD20.1, U19.6 (DIN)
- new net: RD20.2, U20.5 (DO)
- new net: L19.3 (RK), U19.1 (OUTR)
- new net: L19.2 (GK), U19.2 (OUTG)
- new net: L19.1 (BK), U19.3 (OUTB)
- new net: C19.1, R19.2, U19.8 (VDD)
- new net: RD21.1, U20.6 (DIN)
- new net: RD21.2, U21.5 (DO)
- new net: L20.3 (RK), U20.1 (OUTR)
- new net: L20.2 (GK), U20.2 (OUTG)
- new net: L20.1 (BK), U20.3 (OUTB)
- new net: C20.1, R20.2, U20.8 (VDD)
- new net: RD22.1, U21.6 (DIN)
- new net: RD22.2, U22.5 (DO)
- new net: L21.3 (RK), U21.1 (OUTR)
- new net: L21.2 (GK), U21.2 (OUTG)
- new net: L21.1 (BK), U21.3 (OUTB)
- new net: C21.1, R21.2, U21.8 (VDD)
- new net: RD23.1, U22.6 (DIN)
- new net: RD23.2, U23.5 (DO)
- new net: L22.3 (RK), U22.1 (OUTR)
- new net: L22.2 (GK), U22.2 (OUTG)
- new net: L22.1 (BK), U22.3 (OUTB)
- new net: C22.1, R22.2, U22.8 (VDD)
- new net: RD24.1, U23.6 (DIN)
- new net: RD24.2, U24.5 (DO)
- new net: L23.3 (RK), U23.1 (OUTR)
- new net: L23.2 (GK), U23.2 (OUTG)
- new net: L23.1 (BK), U23.3 (OUTB)
- new net: C23.1, R23.2, U23.8 (VDD)
- new net: RD25.1, U24.6 (DIN)
- new net: RD25.2, U25.5 (DO)
- new net: L24.3 (RK), U24.1 (OUTR)
- new net: L24.2 (GK), U24.2 (OUTG)
- new net: L24.1 (BK), U24.3 (OUTB)
- new net: C24.1, R24.2, U24.8 (VDD)
- new net: RD26.1, U25.6 (DIN)
- new net: RD26.2, U26.5 (DO)
- new net: L25.3 (RK), U25.1 (OUTR)
- new net: L25.2 (GK), U25.2 (OUTG)
- new net: L25.1 (BK), U25.3 (OUTB)
- new net: C25.1, R25.2, U25.8 (VDD)
- new net: RD27.1, U26.6 (DIN)
- new net: RD27.2, U27.5 (DO)
- new net: L26.3 (RK), U26.1 (OUTR)
- new net: L26.2 (GK), U26.2 (OUTG)
- new net: L26.1 (BK), U26.3 (OUTB)
- new net: C26.1, R26.2, U26.8 (VDD)
- new net: RD28.1, U27.6 (DIN)
- new net: RD28.2, U28.5 (DO)
- new net: L27.3 (RK), U27.1 (OUTR)
- new net: L27.2 (GK), U27.2 (OUTG)
- new net: L27.1 (BK), U27.3 (OUTB)
- new net: C27.1, R27.2, U27.8 (VDD)
- new net: RD29.1, U28.6 (DIN)
- new net: L28.3 (RK), U28.1 (OUTR)
- new net: L28.2 (GK), U28.2 (OUTG)
- new net: L28.1 (BK), U28.3 (OUTB)
- new net: C28.1, R28.2, U28.8 (VDD)
Other:
- moved on the sheet: RD10, RD105, RD11, RD12, RD13, RD14, RD15, RD16, RD2, RD3, RD30, RD31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

Commit message: Placed and routed second row
Parts:
- added RD17, RDR1: 33R, Resistor_SMD:R_0805_2012Metric, symbol Device:R_Small
Connections:
- net at U17.5 (DO): now also RD17.1
- net at U34.6 (DIN): now also RDR1.1
- net at U16.5 (DO): now also RDR1.2
Changed lines of the file:
@@
 Wire Wire Line
 	1300 12500 1400 12500
+$Comp
+L Device:R_Small RDR1
+U 1 1 5D6BA691
+P 38650 14350
+F 0 "RDR1" V 38501 14350 30  0000 C CNN
+F 1 "33R" V 38561 14350 30  0000 C CNN
+F 2 "Resistor_SMD:R_0805_2012Metric" H 38650 14350 50  0001 C CNN
+F 3 "~" H 38650 14350 50  0001 C CNN
+	1    38650 14350
+	0    1    1    0
+$EndComp
+Wire Wire Line
+	-6100 14450 -6725 14450
+$Comp
+L Device:R_Small RD17
+U 1 1 5DBF44A3
+P -6825 14450
+F 0 "RD17" V -6974 14450 30  0000 C CNN
+F 1 "33R" V -6914 14450 30  0000 C CNN
+F 2 "Resistor_SMD:R_0805_2012Metric" H -6825 14450 50  0001 C CNN
+F 3 "~" H -6825 14450 50  0001 C CNN
+	1    -6825 14450
+	0    1    1    0
+$EndComp
 $EndSCHEMATC

Commit message: Added third RGB row to schematic
Parts:
- removed RD17: 33R, Resistor_SMD:R_0805_2012Metric, symbol Device:R_Small
- added C35, C36, C37, C38, C39, C40, C41, C42, C43, C44, C45, C46, C47, C48, C49, C50, C51: 100nF, Capacitor_SMD:C_0805_2012Metric, symbol Device:C_Small
- added L35, L36, L37, L38, L39, L40, L41, L42, L43, L44, L45, L46, L47, L48, L49, L50, L51: LED_BGRA, acheron_Components:LED_RGB_SMD_6028_2.8x3.5mm_Round, symbol Device:LED_BGRA
- added R35, R36, R37, R38, R39, R40, R41, R42, R43, R44, R45, R46, R47, R48, R49, R50, R51: 100R, Resistor_SMD:R_0805_2012Metric, symbol Device:R_Small
- added RD35, RD36, RD37, RD38, RD39, RD40, RD41, RD42, RD43, RD44, RD45, RD46, RD47, RD48, RD49, RD50, RD51: 33R, Resistor_SMD:R_0805_2012Metric, symbol Device:R_Small
- added U35, U36, U37, U38, U39, U40, U41, U42, U43, U44, U45, U46, U47, U48, U49, U50, U51: WS2811M, acheron_Components:MSOP-8-1EP_3x3mm_P0.65mm_EP1.68x1.88mm, symbol acheronSymbols:WS2811M
Connections:
- net 5V: now also L35.4 (A), L36.4 (A), L37.4 (A), L38.4 (A), L39.4 (A), L40.4 (A), L41.4 (A), L42.4 (A), L43.4 (A), L44.4 (A), L45.4 (A), L46.4 (A), L47.4 (A), L48.4 (A), L49.4 (A), L50.4 (A), L51.4 (A), R35.1, R36.1, R37.1, R38.1, R39.1, R40.1, R41.1, R42.1, R43.1, R44.1, R45.1, R46.1, R47.1, R48.1, R49.1, R50.1, R51.1
- net GND: now also C35.2, C36.2, C37.2, C38.2, C39.2, C40.2, C41.2, C42.2, C43.2, C44.2, C45.2, C46.2, C47.2, C48.2, C49.2, C50.2, C51.2, U35.4 (GND), U35.9 (GND), U36.4 (GND), U36.9 (GND), U37.4 (GND), U37.9 (GND), U38.4 (GND), U38.9 (GND), U39.4 (GND), U39.9 (GND), U40.4 (GND), U40.9 (GND), U41.4 (GND), U41.9 (GND), U42.4 (GND), U42.9 (GND), U43.4 (GND), U43.9 (GND), U44.4 (GND), U44.9 (GND), U45.4 (GND), U45.9 (GND), U46.4 (GND), U46.9 (GND), U47.4 (GND), U47.9 (GND), U48.4 (GND), U48.9 (GND), U49.4 (GND), U49.9 (GND), U50.4 (GND), U50.9 (GND), U51.4 (GND), U51.9 (GND)
- net at U17.5 (DO): now also RD35.2
- new net: L35.3 (RK), U35.1 (OUTR)
- new net: L35.2 (GK), U35.2 (OUTG)
- new net: L35.1 (BK), U35.3 (OUTB)
- new net: RD36.2, U35.5 (DO)
- new net: RD35.1, U35.6 (DIN)
- new net: C35.1, R35.2, U35.8 (VDD)
- new net: L36.3 (RK), U36.1 (OUTR)
- new net: L36.2 (GK), U36.2 (OUTG)
- new net: L36.1 (BK), U36.3 (OUTB)
- new net: RD37.2, U36.5 (DO)
- new net: RD36.1, U36.6 (DIN)
- new net: C36.1, R36.2, U36.8 (VDD)
- new net: L37.3 (RK), U37.1 (OUTR)
- new net: L37.2 (GK), U37.2 (OUTG)
- new net: L37.1 (BK), U37.3 (OUTB)
- new net: RD38.2, U37.5 (DO)
- new net: RD37.1, U37.6 (DIN)
- new net: C37.1, R37.2, U37.8 (VDD)
- new net: L38.3 (RK), U38.1 (OUTR)
- new net: L38.2 (GK), U38.2 (OUTG)
- new net: L38.1 (BK), U38.3 (OUTB)
- new net: RD39.2, U38.5 (DO)
- new net: RD38.1, U38.6 (DIN)
- new net: C38.1, R38.2, U38.8 (VDD)
- new net: L39.3 (RK), U39.1 (OUTR)
- new net: L39.2 (GK), U39.2 (OUTG)
- new net: L39.1 (BK), U39.3 (OUTB)
- new net: RD40.2, U39.5 (DO)
- new net: RD39.1, U39.6 (DIN)
- new net: C39.1, R39.2, U39.8 (VDD)
- new net: L40.3 (RK), U40.1 (OUTR)
- new net: L40.2 (GK), U40.2 (OUTG)
- new net: L40.1 (BK), U40.3 (OUTB)
- new net: RD41.2, U40.5 (DO)
- new net: RD40.1, U40.6 (DIN)
- new net: C40.1, R40.2, U40.8 (VDD)
- new net: L41.3 (RK), U41.1 (OUTR)
- new net: L41.2 (GK), U41.2 (OUTG)
- new net: L41.1 (BK), U41.3 (OUTB)
- new net: RD42.2, U41.5 (DO)
- new net: RD41.1, U41.6 (DIN)
- new net: C41.1, R41.2, U41.8 (VDD)
- new net: L42.3 (RK), U42.1 (OUTR)
- new net: L42.2 (GK), U42.2 (OUTG)
- new net: L42.1 (BK), U42.3 (OUTB)
- new net: RD43.2, U42.5 (DO)
- new net: RD42.1, U42.6 (DIN)
- new net: C42.1, R42.2, U42.8 (VDD)
- new net: L43.3 (RK), U43.1 (OUTR)
- new net: L43.2 (GK), U43.2 (OUTG)
- new net: L43.1 (BK), U43.3 (OUTB)
- new net: RD44.2, U43.5 (DO)
- new net: RD43.1, U43.6 (DIN)
- new net: C43.1, R43.2, U43.8 (VDD)
- new net: L44.3 (RK), U44.1 (OUTR)
- new net: L44.2 (GK), U44.2 (OUTG)
- new net: L44.1 (BK), U44.3 (OUTB)
- new net: RD45.2, U44.5 (DO)
- new net: RD44.1, U44.6 (DIN)
- new net: C44.1, R44.2, U44.8 (VDD)
- new net: L45.3 (RK), U45.1 (OUTR)
- new net: L45.2 (GK), U45.2 (OUTG)
- new net: L45.1 (BK), U45.3 (OUTB)
- new net: RD46.2, U45.5 (DO)
- new net: RD45.1, U45.6 (DIN)
- new net: C45.1, R45.2, U45.8 (VDD)
- new net: L46.3 (RK), U46.1 (OUTR)
- new net: L46.2 (GK), U46.2 (OUTG)
- new net: L46.1 (BK), U46.3 (OUTB)
- new net: RD47.2, U46.5 (DO)
- new net: RD46.1, U46.6 (DIN)
- new net: C46.1, R46.2, U46.8 (VDD)
- new net: RD47.1, U47.6 (DIN)
- new net: L47.3 (RK), U47.1 (OUTR)
- new net: L47.2 (GK), U47.2 (OUTG)
- new net: L47.1 (BK), U47.3 (OUTB)
- new net: RD48.2, U47.5 (DO)
- new net: C47.1, R47.2, U47.8 (VDD)
- new net: RD48.1, U48.6 (DIN)
- new net: L48.3 (RK), U48.1 (OUTR)
- new net: L48.2 (GK), U48.2 (OUTG)
- new net: L48.1 (BK), U48.3 (OUTB)
- new net: RD49.2, U48.5 (DO)
- new net: C48.1, R48.2, U48.8 (VDD)
- new net: RD49.1, U49.6 (DIN)
- new net: L49.3 (RK), U49.1 (OUTR)
- new net: L49.2 (GK), U49.2 (OUTG)
- new net: L49.1 (BK), U49.3 (OUTB)
- new net: RD50.2, U49.5 (DO)
- new net: C49.1, R49.2, U49.8 (VDD)
- new net: RD50.1, U50.6 (DIN)
- new net: L50.3 (RK), U50.1 (OUTR)
- new net: L50.2 (GK), U50.2 (OUTG)
- new net: L50.1 (BK), U50.3 (OUTB)
- new net: RD51.2, U50.5 (DO)
- new net: C50.1, R50.2, U50.8 (VDD)
- new net: RD51.1, U51.6 (DIN)
- new net: L51.3 (RK), U51.1 (OUTR)
- new net: L51.2 (GK), U51.2 (OUTG)
- new net: L51.1 (BK), U51.3 (OUTB)
- new net: C51.1, R51.2, U51.8 (VDD)

Commit message: Routed 3rd row and columns
- The RGB 3rd row was routed; all components were added, their labels fixed and cleaned.
- All columns were routed. Some were reassigned for better fitting. It may be that I'll redo some columns in the near future as the routing does not look clean, specially in the bottom row;
- A warning sign was added to show that, when using a screw-in stab on the 2U backspace, there should be an electric tape preventing the screw from short-circuiting to the column pad.
Parts:
- added G3: Warning sign, acheron_Graphics:warning_sign_3.6x3.2mm, symbol Mechanical:MountingHole
Connections:
- net Col10: now also SW8.1 (Col); no longer SW9.1 (Col)
- net Col11: now also SW9.1 (Col)
- net Col12: no longer SW100.1 (Col), SW84.1 (Col)
- net Col13: now also SW100.1 (Col), SW84.1 (Col)
- net Col7: no longer SW6.1 (Col)
- net Col8: now also SW6.1 (Col); no longer SW7.1 (Col)
- net Col9: now also SW7.1 (Col); no longer SW8.1 (Col)
Other:
- moved on the sheet: C1, C10, C105, C11, C12, C13, C14, C15, C16, C17, C18, C19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
