File: PCB Files/TKL.kicad_pcb (KiCad board)
At the start: 2 copper layers, 350 x 123.8 mm, 557 parts, among them J1 USB_C, SW1 ESC, SW10 F9, SW100 RGUI_R2, SW101 RCTRL_R2, SW102 STEPPED_CAPS, SW103 RSHFT_175, SW104 Fn, SW105 BKSP_2U, SW11 F10, SW12 F11, SW13 F12, SW14 PRTSC, SW15 SCRLCK, SW16 PAUSE, SW17 GRV, SW18 1, SW19 2, SW2 F1, SW20 3, SW21 4, SW22 5, SW23 6, SW24 7, SW25 8, SW26 9, SW27 0, SW28 HIFEN, SW29 PLUS, SW3 F2, SW30 BCKSLSH, SW31 DEL, SW32 INS, SW33 HOME, SW34 PGUP, SW35 TAB, SW36 Q, SW37 W, SW38 E, SW39 R, SW4 F3, SW40 T, SW41 Y, SW42 U, SW43 I, SW44 O, SW45 P, SW46 LBRACES, SW47 RBRACES, SW48 BKSP_150, SW49 DEL, SW5 F4, SW50 END, SW51 PGDN, SW52 CAPS, SW53 A, SW54 S, SW55 D, SW56 F, SW57 G, SW58 H, SW59 J, SW6 F5, SW60 K, SW61 L, SW62 :, SW63 QUOTE, SW64 ENTER, SW65 LSHFT, SW66 Z, SW67 X, SW68 C, SW69 V, SW7 F6, SW70 B, SW71 N, SW72 M, SW73 <,, SW74 .>, SW75 /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

Commit message: Routed SW57 RGB LED
Parts:
- moved C57 294.5 mm to (329.8, 122.8)
- moved R57 270.2 mm to (329.8, 120.7), turned to 180 degrees
- moved RD56 266.2 mm to (329.8, 124.8)
Routing:
- net Net-(L57-Pad1): track 0.00 -> 16.6 mm
- net Net-(RD54-Pad1): track 33.2 -> 49.8 mm
- net Net-(L57-Pad2): track 0.00 -> 7.72 mm
- net 5V: track 2039.1 -> 2043.8 mm, vias 60 -> 61
- net Net-(L57-Pad3): track 0.00 -> 4.39 mm
- net Net-(C57-Pad1): track 0.00 -> 3.84 mm
- net Net-(RD54-Pad2): track 3.93 -> 5.90 mm

Commit message: Routed SW58 RGB LED
Parts:
- moved C58 286.3 mm to (310.7, 122.8)
- moved RD57 247.1 mm to (310.7, 124.8)
- moved R58 232.1 mm to (310.7, 120.7), turned to 180 degrees
Routing:
- net Net-(L58-Pad1): track 0.00 -> 16.6 mm
- net Net-(RD54-Pad1): track 49.8 -> 66.4 mm
- net Net-(L58-Pad2): track 0.00 -> 7.72 mm
- net 5V: track 2043.8 -> 2048.5 mm, vias 61 -> 62
- net Net-(L58-Pad3): track 0.00 -> 4.39 mm
- net Net-(C58-Pad1): track 0.00 -> 3.84 mm
- net Net-(RD54-Pad2): track 5.90 -> 7.87 mm

Commit message: Routed SW59 RGB LED
Parts:
- moved C59 265.3 mm to (291.7, 122.8)
- moved R59 220.0 mm to (291.7, 120.7), turned to 180 degrees
- moved RD58 219.4 mm to (291.7, 124.8), turned to 180 degrees
Routing:
- net 5V: track 2048.5 -> 2095.2 mm, vias 62 -> 63
- net Net-(L59-Pad1): track 0.00 -> 16.6 mm
- net Net-(RD58-Pad1): track 0.00 -> 16.6 mm
- net Net-(L59-Pad2): track 0.00 -> 7.72 mm
- net Net-(L59-Pad3): track 0.00 -> 4.39 mm
- net Net-(C59-Pad1): track 0.00 -> 3.84 mm
- net Net-(RD58-Pad2): track 0.00 -> 1.97 mm
- net Col6: track 104.1 -> 105.0 mm
