File: PCB Files/TKL.kicad_pcb (KiCad board)
At the start: 2 copper layers, 350 x 123.8 mm, 557 parts, among them J1 USB_C, SW1 ESC, SW10 F9, SW100 RGUI_R2, SW101 RCTRL_R2, SW102 STEPPED_CAPS, SW103 RSHFT_175, SW104 Fn, SW105 BKSP_2U, SW11 F10, SW12 F11, SW13 F12, SW14 PRTSC, SW15 SCRLCK, SW16 PAUSE, SW17 GRV, SW18 1, SW19 2, SW2 F1, SW20 3, SW21 4, SW22 5, SW23 6, SW24 7, SW25 8, SW26 9, SW27 0, SW28 HIFEN, SW29 PLUS, SW3 F2, SW30 BCKSLSH, SW31 DEL, SW32 INS, SW33 HOME, SW34 PGUP, SW35 TAB, SW36 Q, SW37 W, SW38 E, SW39 R, SW4 F3, SW40 T, SW41 Y, SW42 U, SW43 I, SW44 O, SW45 P, SW46 LBRACES, SW47 RBRACES, SW48 BKSP_150, SW49 DEL, SW5 F4, SW50 END, SW51 PGDN, SW52 CAPS, SW53 A, SW54 S, SW55 D, SW56 F, SW57 G, SW58 H, SW59 J, SW6 F5, SW60 K, SW61 L, SW62 :, SW63 QUOTE, SW64 ENTER, SW65 LSHFT, SW66 Z, SW67 X, SW68 C, SW69 V, SW7 F6, SW70 B, SW71 N, SW72 M, SW73 <,, SW74 .>, SW75 /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

Commit message: Routed SW60 RGB LED
Parts:
- moved C60 230.5 mm to (272.6, 122.8)
- moved RD59 201.0 mm to (272.6, 124.8), turned to 180 degrees
- moved R60 200.4 mm to (272.6, 120.7), turned to 180 degrees
Routing:
- net 5V: track 2095.2 -> 2121.0 mm, vias 63 -> 64
- net Net-(L60-Pad1): track 0.00 -> 16.6 mm
- net Net-(RD59-Pad1): track 0.00 -> 16.6 mm
- net Net-(L60-Pad2): track 0.00 -> 7.72 mm
- net Net-(L60-Pad3): track 0.00 -> 4.39 mm
- net Net-(C60-Pad1): track 0.00 -> 3.84 mm
- net Net-(RD59-Pad2): track 0.00 -> 1.97 mm

Commit message: Routed SW61 RGB LED
Parts:
- moved C61 217.7 mm to (253.6, 122.8)
- moved RD60 199.6 mm to (253.6, 124.8), turned to 180 degrees
- moved R61 172.5 mm to (253.6, 120.7), turned to 180 degrees
Routing:
- net 5V: track 2121.0 -> 2146.7 mm, vias 64 -> 65
- net Net-(L61-Pad1): track 0.00 -> 16.6 mm
- net Net-(RD60-Pad1): track 0.00 -> 16.6 mm
- net Net-(L61-Pad2): track 0.00 -> 7.72 mm
- net Net-(L61-Pad3): track 0.00 -> 4.39 mm
- net Col13: track 270.7 -> 266.7 mm
- net Net-(C61-Pad1): track 0.00 -> 3.84 mm
- net Net-(RD60-Pad2): track 0.00 -> 1.97 mm

Commit message: Routed SW62 RGB LED
Parts:
- moved C62 215.3 mm to (234.5, 122.8)
- moved R62 169.7 mm to (234.5, 120.7), turned to 180 degrees
- moved RD61 157.7 mm to (234.5, 124.8), turned to 180 degrees
Routing:
- net 5V: track 2146.7 -> 2172.4 mm, vias 65 -> 66
- net Net-(L62-Pad1): track 0.00 -> 16.6 mm
- net Net-(RD61-Pad1): track 0.00 -> 16.6 mm
- net Net-(L62-Pad2): track 0.00 -> 7.72 mm
- net Net-(L62-Pad3): track 0.00 -> 4.39 mm
- net Net-(C62-Pad1): track 0.00 -> 3.84 mm
- net Net-(RD61-Pad2): track 0.00 -> 1.97 mm
